File: PCB/PWR/PWR.kicad_pcb (KiCad board)
At the start: 2 copper layers, 40 x 46.2 mm, 44 parts, among them IC1 SN74LVC2G00DCURE4, J1 switch, J2 Conn_02x06_Odd_Even, J3 Battery, U1 AP2112K-3.3, U2 BQ25570, U3 AP2112K-1.8, U4 MCP73831-2-OT

Commit message: udated by FZ from Windows
Parts:
- added J4: Solar cell, Connector_PinHeader_2.00mm:PinHeader_2x01_P2.00mm_Vertical, F.Cu at (165.0, 92.0)
- moved J3 34.2 mm to (165.0, 99.0), turned to 90 degrees
- moved D1 23.7 mm to (157.6, 99.7)
- moved R16 20.6 mm to (153.5, 99.6), turned to 180 degrees
- moved C13 20.6 mm to (157.0, 103.6)
- moved C4 20.6 mm to (150.0, 102.4)
- moved R15 20.6 mm to (157.5, 101.4)
- moved U4 20.6 mm to (153.5, 102.4)
- moved TP4 15.1 mm to (140.3, 107.2)
- moved TP3 10.3 mm to (151.7, 80.9)
- moved C1 7.14 mm to (150.4, 108.5), turned to 0 degrees
- moved R3 6.01 mm to (144.2, 110.7), turned to 90 degrees
- moved R2 5.98 mm to (150.4, 107.3), turned to 0 degrees
- moved IC1 5.79 mm to (149.3, 110.7), turned to 0 degrees
- moved R4 5.67 mm to (145.5, 110.8), turned to 90 degrees
- moved C12 5.07 mm to (136.5, 103.3)
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Connections:
- J2 pad 1: +5V -> /VBAT_OK
- J2 pad 10: /VBAT_OK -> +1V8
- J2 pad 12: GND -> +5V
- J2 pad 2: /VBAT -> /~{EN}
- J2 pad 3: /SC -> unconnected-(J2-Pad3)
- J2 pad 4: /SC -> unconnected-(J2-Pad4)
- J2 pad 5: +3V3 -> unconnected-(J2-Pad5)
- J2 pad 6: +3V3 -> /VBAT
- J2 pad 7: +1V8 -> +3V3
- J2 pad 8: unconnected-(J2-Pad8) -> +3V3
- J2 pad 9: /~{EN} -> +1V8
Routing:
- net /VBAT: track 0.00 -> 82.2 mm, vias 0 -> 4
- net +5V: track 0.00 -> 38.1 mm, vias 0 -> 3
- net /SC: track 0.00 -> 27.6 mm
- net /VBAT_OK: track 2.59 -> 27.7 mm
- net /PWR_EN: track 0.00 -> 20.6 mm
- net /~{EN}: track 9.13 -> 23.6 mm
- net +1V8: track 0.00 -> 13.8 mm
- net Net-(C1-Pad1): track 0.00 -> 12.8 mm, vias 0 -> 1
- net +3V3: track 0.00 -> 11.0 mm
- net Net-(C6-Pad1): track 7.74 -> 14.8 mm
- net Net-(C1-Pad2): track 0.00 -> 6.76 mm
- net Net-(D1-Pad1): track 0.00 -> 4.90 mm
- net Net-(C5-Pad1): track 0.00 -> 4.80 mm
- net Net-(R16-Pad1): track 0.00 -> 2.80 mm
- net Net-(R15-Pad2): track 0.00 -> 1.95 mm
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- added copper zone on B.Cu, net GND
- added copper zone on F.Cu, net GND

Commit message: udated by FZ from Windows
Connections:
- J2 pad 1: /VBAT_OK -> GND
- J2 pad 3: unconnected-(J2-Pad3) -> GND
- J2 pad 4: unconnected-(J2-Pad4) -> /VBAT_OK
- J2 pad 5: unconnected-(J2-Pad5) -> GND
Routing:
- net /VBAT_OK: track 27.7 -> 24.1 mm
