File: PCB/PWR/PWR.kicad_sch (KiCad schematic)
At the start: 1 part

Commit message: udated by FZ from Windows
Parts:
- added C1, C5: (no value), symbol Device:C_Small
- added C10: 47uF, symbol Device:C_Polarized_Small_US
- added C11, C13, C2, C9: 0.1uF, symbol Device:C_Small
- added C12: (no value), symbol Device:C_Polarized_Small_US
- added C3, C4: 4.7uF, symbol Device:C_Small
- added C6: 22uF, symbol Device:C_Small
- added C7: 10uF, symbol Device:C_Small
- added C8: 0.01uF, symbol Device:C_Small
- added D1: RED, symbol Device:LED_Small_Filled
- added IC1: (no value), symbol SamacSys_Parts:SN74LVC2G00DCURE4
- added J1, J3: (no value), symbol Connector:Conn_01x02_Male
- added J2: (no value), symbol Connector_Generic:Conn_02x06_Odd_Even
- added L1: 4.7uH, symbol Device:L_Small
- added L2: 22uH, symbol Device:L_Small
- added R1, R16, R2, R3, R4, R5: (no value), symbol Device:R_Small
- added R10, R11, R14, R15, R6, R7, R8, R9: 1k, symbol Device:R_Small
- added R12, R13: 10k, symbol Device:R_Small
- added TP1, TP2, TP3, TP4: TestPoint_Alt, symbol Connector:TestPoint_Alt
- added U1: AP2112K-3.3, Package_TO_SOT_SMD:SOT-23-5, symbol Regulator_Linear:AP2112K-3.3
- added U3: (no value), symbol Regulator_Linear:AP2112K-1.8
- added U4: MCP73831-2-OT, Package_TO_SOT_SMD:SOT-23-5, symbol Battery_Management:MCP73831-2-OT
- gave numbers to parts that had none: 1
Connections:
- net GND: now reaches U2.1 (VSS), U2.15 (VSS), U2.17 (VSS), U2.21 (VSS), U2.9 (VSS)
- net GND: now also C10.2, C11.2, C12.2, C13.2, C2.2, C3.2, C4.2, C5.2, C6.2, C7.2, C8.2, C9.2, IC1.4 (GND), J1.2 (Pin_2), J2.11 (Pin_11), J2.12 (Pin_12), J3.2 (Pin_2), R11.1, R12.1, R13.1, R14.1, R15.1, R3.1, R4.1, R9.1, U1.2 (GND), U3.2 (GND), U4.2 (VSS)
- net at U2.10 (OK_HYST): now also R10.2, R7.1
- net at U2.11 (OK_PROG): now also R10.1, R14.2
- net at U2.12 (VOUT_SET): now also R11.2, R8.1
- net VBAT_OK: now reaches U2.13 (VBAT_OK)
- net VBAT_OK: now also J2.10 (Pin_10)
- net at U2.14 (VOUT): now also C6.1, L1.2, TP2.1
- net at U2.16 (LBUCK): now also L1.1
- net VBAT: now reaches U2.18 (VBAT)
- net VBAT: now also C11.1, C4.1, C9.1, IC1.8 (VCC), J2.2 (Pin_2), J3.1 (Pin_1), R1.2, R2.2, TP1.1, U1.1 (VIN), U3.1 (VIN), U4.3 (VBAT)
- net at U2.19 (VSTOR): now also U2.3 (VOC_SAMP), C2.1, C3.1
- net SC: now reaches U2.2 (VIN_DC)
- net SC: now also C7.1, J2.3 (Pin_3), J2.4 (Pin_4), L2.1, TP3.1
- net at U2.20 (LBOOST): now also L2.2
- net at U2.4 (VREF_SAMP): now also C8.1
- net ~{EN}: now reaches U2.5 (~{EN})
- net ~{EN}: now also J2.9 (Pin_9), R13.2
- net VOUT_EN: now reaches U2.6 (VOUT_EN)
- net VOUT_EN: now also R12.2
- net at U2.7 (VBAT_OV): now also R6.1, R9.2
- net at U2.8 (VRDIV): now also R6.2, R7.2, R8.2
- new net: C1.2, IC1.5 (2A), R2.1
- new net: C5.1, IC1.1 (1A), R5.1
- new net: C1.1, J1.1 (Pin_1), R1.1, R5.2
- new net: IC1.6 (2B), IC1.7 (1Y)
- new net: R16.1, U4.1 (STAT)
- new net: D1.1 (K), R16.2
- new net: R15.2, U4.5 (PROG)
- new net +1V8: C12.1, J2.7 (Pin_7), U3.5 (VOUT)
- new net +3V3: C10.1, J2.5 (Pin_5), J2.6 (Pin_6), U1.5 (VOUT)
- new net +5V: C13.1, D1.2 (A), J2.1 (Pin_1), TP4.1, U4.4 (VDD)
- new net PWR_EN: IC1.2 (1B), IC1.3 (2Y), R3.2, R4.2, U1.3 (EN), U3.3 (EN)
Other:
- note added: "BQ25570"
- note added: "Connectors"
- note added: "Li-Ion charger"
- note added: "Mounting holes"
- note added: "Power supply"
- note added: "Solar cell: KXOB201K04F-TR or SM111K04L"
- note added: "Switch circuit"
- note added: "http://www.mosaic-industries.com/embedded-systems/microcontroller-projects/electronic-circuits/push-button-switch-turn-on/ latching-toggle-power-switch#press-on-hold-off-latching-circuits"
- company: (none) -> MIT Media Lab
- title: (none) -> HexSense Svalbard - PWR
- moved on the sheet: U2

Commit message: udated by FZ from Windows
Parts:
- added J4: (no value), Connector_PinHeader_2.00mm:PinHeader_2x01_P2.00mm_Vertical, symbol Connector:Conn_01x02_Male
- C1, C5: value (none) -> 1uF; footprint (none) -> Capacitor_SMD:C_0402_1005Metric_Pad0.74x0.62mm_HandSolder
- C10: footprint (none) -> LED_SMD:LED_0805_2012Metric_Pad1.15x1.40mm_HandSolder
- C11, C13, C2, C8, C9: footprint (none) -> Capacitor_SMD:C_0402_1005Metric_Pad0.74x0.62mm_HandSolder
- C12: value (none) -> 47uF; footprint (none) -> LED_SMD:LED_0805_2012Metric_Pad1.15x1.40mm_HandSolder
- C3, C4, C7: footprint (none) -> Capacitor_SMD:C_0603_1608Metric_Pad1.08x0.95mm_HandSolder
- C6: footprint (none) -> Capacitor_SMD:C_0805_2012Metric_Pad1.18x1.45mm_HandSolder
- D1: footprint (none) -> LED_SMD:LED_0603_1608Metric_Pad1.05x0.95mm_HandSolder
- IC1: value (none) -> SN74LVC2G00DCURE4; footprint (none) -> SOP50P310X90-8N
- J1: value (none) -> switch; footprint (none) -> Connector_PinHeader_2.54mm:PinHeader_1x02_P2.54mm_Vertical
- J2: value (none) -> Conn_02x06_Odd_Even; footprint (none) -> Connector_PinHeader_2.54mm:PinHeader_2x06_P2.54mm_Vertical
- J3: value (none) -> Battery; footprint (none) -> Connector_PinHeader_2.00mm:PinHeader_2x01_P2.00mm_Vertical
- L1: footprint (none) -> Inductor_SMD:L_Wuerth_MAPI-3015
- L2: footprint (none) -> Inductor_SMD:L_Taiyo-Yuden_NR-40xx_HandSoldering
- R1, R2: value (none) -> 100k; footprint (none) -> Resistor_SMD:R_0402_1005Metric_Pad0.72x0.64mm_HandSolder
- R10, R11, R12, R13, R14, R15, R6, R7, R8, R9: footprint (none) -> Resistor_SMD:R_0603_1608Metric_Pad0.98x0.95mm_HandSolder
- R16: value (none) -> 100; footprint (none) -> Resistor_SMD:R_0603_1608Metric_Pad0.98x0.95mm_HandSolder
- R3, R4: value (none) -> NC; footprint (none) -> Resistor_SMD:R_0402_1005Metric_Pad0.72x0.64mm_HandSolder
- R5: value (none) -> 1M; footprint (none) -> Resistor_SMD:R_0603_1608Metric_Pad0.98x0.95mm_HandSolder
- TP1, TP2, TP3, TP4: footprint (none) -> TestPoint:TestPoint_Pad_1.0x1.0mm
- U3: value (none) -> AP2112K-1.8; footprint (none) -> Package_TO_SOT_SMD:SOT-23-5
Connections:
- net +1V8: now also J2.10 (Pin_10), J2.9 (Pin_9); no longer J2.7 (Pin_7)
- net +3V3: now also J2.7 (Pin_7), J2.8 (Pin_8); no longer J2.5 (Pin_5), J2.6 (Pin_6)
- net +5V: now also J2.12 (Pin_12); no longer J2.1 (Pin_1)
- net GND: now also J4.2 (Pin_2); no longer J2.12 (Pin_12)
- net SC: now also J4.1 (Pin_1); no longer J2.3 (Pin_3), J2.4 (Pin_4)
- net VBAT: now also J2.6 (Pin_6); no longer J2.2 (Pin_2)
- net VBAT_OK: now also J2.1 (Pin_1); no longer J2.10 (Pin_10)
- net ~{EN}: now also J2.2 (Pin_2); no longer J2.9 (Pin_9)
Other:
- moved on the sheet: C2, C3, C4, C6, C7, C8, J3, L1, L2, R10, R11, R12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

Commit message: udated by FZ from Windows
Parts:
- J4: value (none) -> Solar cell
Connections:
- net GND: now also J2.1 (Pin_1), J2.3 (Pin_3), J2.5 (Pin_5)
- net VBAT_OK: now also J2.4 (Pin_4); no longer J2.1 (Pin_1)
Changed lines of the file:
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@@
-    (stroke (width 0) (type default) (color 0 0 0 0))
-  )
-  (wire (pts (xy 142.24 69.85) (xy 151.13 69.85))
     (stroke (width 0) (type default) (color 0 0 0 0))
   )
@@
     (stroke (width 0) (type default) (color 0 0 0 0))
   )
-  (wire (pts (xy 142.24 72.39) (xy 151.13 72.39))
+  (wire (pts (xy 144.78 72.39) (xy 151.13 72.39))
     (stroke (width 0) (type default) (color 0 0 0 0))
   )
@@
     (stroke (width 0) (type default) (color 0 0 0 0))
   )
+  (wire (pts (xy 144.78 69.85) (xy 151.13 69.85))
+    (stroke (width 0) (type default) (color 0 0 0 0))
+  )
   (wire (pts (xy 96.52 73.66) (xy 109.22 73.66))
     (stroke (width 0) (type default) (color 0 0 0 0))
@@
     (stroke (width 0) (type default) (color 0 0 0 0))
   )
-  (wire (pts (xy 142.24 74.93) (xy 151.13 74.93))
+  (wire (pts (xy 144.78 74.93) (xy 151.13 74.93))
     (stroke (width 0) (type default) (color 0 0 0 0))
   )
@@
     (effects (font (size 1.27 1.27)) (justify right bottom))
   )
-  (label "VBAT_OK" (at 142.24 69.85 0)
-    (effects (font (size 1.27 1.27)) (justify left bottom))
+  (label "VBAT_OK" (at 172.72 72.39 180)
+    (effects (font (size 1.27 1.27)) (justify right bottom))
   )
   (label "PWR_EN" (at 200.66 92.71 0)
@@
     (pin "1")
   )
+  (symbol (lib_id "power:GND") (at 144.78 69.85 270) (unit 1)
+    (in_bom yes) (on_board yes)
+    (property "Reference" "#PWR0126" (id 0) (at 138.43 69.85 0)
+      (effects (font (size 1.27 1.27)) hide)
+    )
+    (property "Value" "GND" (id 1) (at 137.16 69.85 90)
+      (effects (font (size 1.27 1.27)) (justify left))
+    )
+    (property "Footprint" "" (id 2) (at 144.78 69.85 0)
+      (effects (font (size 1.27 1.27)) hide)
+    )
+    (property "Datasheet" "" (id 3) (at 144.78 69.85 0)
+      (effects (font (size 1.27 1.27)) hide)
+    )
+    (pin "1")
+  )
   (symbol (lib_id "Device:R_Small") (at 45.72 92.71 180) (unit 1)
     (in_bom yes) (on_board yes)
@@
     (pin "1")
   )
+  (symbol (lib_id "power:GND") (at 144.78 74.93 270) (unit 1)
+    (in_bom yes) (on_board yes)
+    (property "Reference" "#PWR0124" (id 0) (at 138.43 74.93 0)
+      (effects (font (size 1.27 1.27)) hide)
+    )
+    (property "Value" "GND" (id 1) (at 137.16 74.93 90)
+      (effects (font (size 1.27 1.27)) (justify left))
+    )
+    (property "Footprint" "" (id 2) (at 144.78 74.93 0)
+      (effects (font (size 1.27 1.27)) hide)
+    )
+    (property "Datasheet" "" (id 3) (at 144.78 74.93 0)
+      (effects (font (size 1.27 1.27)) hide)
+    )
+    (pin "1")
+  )
   (symbol (lib_id "Device:C_Small") (at 31.75 62.23 0) (unit 1)
     (in_bom yes) (on_board yes)
@@
     (pin "1")
   )
+  (symbol (lib_id "power:GND") (at 144.78 72.39 270) (unit 1)
+    (in_bom yes) (on_board yes)
+    (property "Reference" "#PWR0125" (id 0) (at 138.43 72.39 0)
+      (effects (font (size 1.27 1.27)) hide)
+    )
+    (property "Value" "GND" (id 1) (at 137.16 72.39 90)
+      (effects (font (size 1.27 1.27)) (justify left))
+    )
+    (property "Footprint" "" (id 2) (at 144.78 72.39 0)
+      (effects (font (size 1.27 1.27)) hide)
+    )
+    (property "Datasheet" "" (id 3) (at 144.78 72.39 0)
+      (effects (font (size 1.27 1.27)) hide)
+    )
+    (pin "1")
+  )
   (symbol (lib_id "Device:R_Small") (at 146.05 33.02 180) (unit 1)
     (in_bom yes) (on_board yes)
@@
     (in_bom yes) (on_board yes)
     (property "Reference" "J4" (id 0) (at 137.16 95.25 0))
-    (property "Value" "" (id 1) (at 138.43 97.79 0))
+    (property "Value" "Solar cell" (id 1) (at 138.43 97.79 0))
     (property "Footprint" "Connector_PinHeader_2.00mm:PinHeader_2x01_P2.00mm_Vertical" (id 2) (at 143.51 96.52 0)
       (effects (font (size 1.27 1.27)) hide)
@@
       (reference "#PWR0123") (unit 1) (value "GND") (footprint "")
     )
+    (path "/5c64e8e8-6c2d-483f-aafc-e21e16486282"
+      (reference "#PWR0124") (unit 1) (value "GND") (footprint "")
+    )
+    (path "/888ac93d-9fbc-4684-9259-e893288eb2ff"
+      (reference "#PWR0125") (unit 1) (value "GND") (footprint "")
+    )
+    (path "/273bb3e6-4d50-47f7-8edd-3059b9c5cc06"
+      (reference "#PWR0126") (unit 1) (value "GND") (footprint "")
+    )
     (path "/f2d1fe8c-a605-48ca-bd7f-38a5ecb369fd"

Commit message: udated by FZ from Windows
Parts:
- IC1: value SN74LVC2G00DCURE4 -> (none)
Connections:
- net GND: no longer J4.2 (Pin_2)
- net SC: now also J4.2 (Pin_2)
Changed lines of the file:
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@@
   (junction (at 96.52 73.66) (diameter 0) (color 0 0 0 0)
   )
-  (junction (at 179.07 101.6) (diameter 0) (color 0 0 0 0)
-  )
   (junction (at 195.58 90.17) (diameter 0) (color 0 0 0 0)
   )
@@
     (stroke (width 0) (type default) (color 0 0 0 0))
   )
+  (wire (pts (xy 152.4 96.52) (xy 152.4 99.06))
+    (stroke (width 0) (type default) (color 0 0 0 0))
+  )
   (wire (pts (xy 195.58 64.77) (xy 209.55 64.77))
     (stroke (width 0) (type default) (color 0 0 0 0))
@@
     (stroke (width 0) (type default) (color 0 0 0 0))
   )
-  (wire (pts (xy 152.4 99.06) (xy 152.4 101.6))
-    (stroke (width 0) (type default) (color 0 0 0 0))
-  )
   (wire (pts (xy 195.58 72.39) (xy 195.58 76.2))
     (stroke (width 0) (type default) (color 0 0 0 0))
@@
   )
   (wire (pts (xy 96.52 81.28) (xy 96.52 82.55))
-    (stroke (width 0) (type default) (color 0 0 0 0))
-  )
-  (wire (pts (xy 152.4 101.6) (xy 179.07 101.6))
     (stroke (width 0) (type default) (color 0 0 0 0))
   )
@@
     (in_bom yes) (on_board yes)
     (property "Reference" "IC1" (id 0) (at 207.01 44.45 0))
-    (property "Value" "SN74LVC2G00DCURE4" (id 1) (at 205.74 29.21 0))
+    (property "Value" "" (id 1) (at 205.74 29.21 0))
     (property "Footprint" "SOP50P310X90-8N" (id 2) (at 236.22 7.62 0)
       (effects (font (size 1.27 1.27)) (justify left) hide)

Commit message: udated by FZ from Windows
Parts:
- IC1: value (none) -> SN74LVC2G00DCURE4
