File: PCB/GEOPHONE_FE/GEOPHONE_FE.kicad_pcb (KiCad board)
At the start: 2 copper layers, 40 x 46.2 mm, 45 parts, among them IC1 SN74LVC2G00DCURE4, J1 switch, J2 Conn_02x06_Odd_Even, J3 Battery, J4 Solar cell, U1 AP2112K-3.3, U2 BQ25570, U3 AP2112K-1.8, U4 MCP73831-2-OT

Commit message: udated by FZ from Windows
Parts:
- removed C1, C5: 1uF, Capacitor_SMD:C_0402_1005Metric_Pad0.74x0.62mm_HandSolder
- removed C10, C12: 47uF, LED_SMD:LED_0805_2012Metric_Pad1.15x1.40mm_HandSolder
- removed C11, C13, C2, C9: 0.1uF, Capacitor_SMD:C_0402_1005Metric_Pad0.74x0.62mm_HandSolder
- removed C3, C4: 4.7uF, Capacitor_SMD:C_0603_1608Metric_Pad1.08x0.95mm_HandSolder
- removed C6: 22uF, Capacitor_SMD:C_0805_2012Metric_Pad1.18x1.45mm_HandSolder
- removed C7: 10uF, Capacitor_SMD:C_0603_1608Metric_Pad1.08x0.95mm_HandSolder
- removed C8: 0.01uF, Capacitor_SMD:C_0402_1005Metric_Pad0.74x0.62mm_HandSolder
- removed D1: RED, LED_SMD:LED_0603_1608Metric_Pad1.05x0.95mm_HandSolder
- removed IC1: SN74LVC2G00DCURE4, Mylib:SOP50P310X90-8N
- removed J1: switch, Connector_PinHeader_2.54mm:PinHeader_1x02_P2.54mm_Vertical
- removed L1: 4.7uH, Inductor_SMD:L_Wuerth_MAPI-3015
- removed L2: 22uH, Inductor_SMD:L_Taiyo-Yuden_NR-40xx_HandSoldering
- removed R1, R2: 100k, Resistor_SMD:R_0402_1005Metric_Pad0.72x0.64mm_HandSolder
- removed R10, R11, R14, R15, R6, R7, R8, R9: 1k, Resistor_SMD:R_0603_1608Metric_Pad0.98x0.95mm_HandSolder
- removed R12, R13: 10k, Resistor_SMD:R_0603_1608Metric_Pad0.98x0.95mm_HandSolder
- removed R16: 100, Resistor_SMD:R_0603_1608Metric_Pad0.98x0.95mm_HandSolder
- removed R3, R4: NC, Resistor_SMD:R_0402_1005Metric_Pad0.72x0.64mm_HandSolder
- removed R5: 1M, Resistor_SMD:R_0603_1608Metric_Pad0.98x0.95mm_HandSolder
- removed TP1, TP2, TP3, TP4: TestPoint_Alt, TestPoint:TestPoint_Pad_1.0x1.0mm
- removed U1: AP2112K-3.3, Package_TO_SOT_SMD:SOT-23-5
- removed U2: BQ25570, Package_DFN_QFN:QFN-20-1EP_3.5x3.5mm_P0.5mm_EP2x2mm
- removed U3: AP2112K-1.8, Package_TO_SOT_SMD:SOT-23-5
- removed U4: MCP73831-2-OT, Package_TO_SOT_SMD:SOT-23-5
Routing:
- net /VBAT: track 82.2 -> 0.00 mm, vias 4 -> 0
- net +5V: track 38.1 -> 0.00 mm, vias 3 -> 0
- net /SC: track 29.8 -> 0.00 mm
- net /VBAT_OK: track 24.1 -> 0.00 mm, vias 1 -> 0
- net /~{EN}: track 23.6 -> 0.00 mm, vias 2 -> 0
- net /PWR_EN: track 20.6 -> 0.00 mm
- net Net-(C6-Pad1): track 14.8 -> 0.00 mm
- net Net-(C2-Pad1): track 14.3 -> 0.00 mm, vias 2 -> 0
- net Net-(R6-Pad2): track 14.0 -> 0.00 mm, vias 3 -> 0
- net +1V8: track 13.8 -> 0.00 mm
- net Net-(C1-Pad1): track 12.8 -> 0.00 mm, vias 1 -> 0
- net +3V3: track 11.0 -> 0.00 mm
- net Net-(R10-Pad1): track 8.28 -> 0.00 mm
- net /VOUT_EN: track 7.89 -> 0.00 mm, vias 2 -> 0
- net Net-(C8-Pad1): track 7.73 -> 0.00 mm
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Other:
- board text removed: "HEXSENSE SVALBARD PWR_V1 FANGZHENG LIU MIT MEDIA LAB ResEnv"
