File: PCB/ADXL355/ADXL355.kicad_pcb (KiCad board)
At the start: 2 copper layers, 40 x 46.2 mm, 10 parts, among them J1 Conn_02x06_Odd_Even, J2 Conn_02x06_Odd_Even, J3 P1, J4 P2, J5 P3

Commit message: udated by FZ from Windows
Connections:
- J1 pad 7: unconnected-(J1-Pad7) -> /RXD
- J1 pad 9: unconnected-(J1-Pad9) -> /TXD
