File: PCB/ADXL355/ADXL355.kicad_sch (KiCad schematic)
At the start: 10 parts, among them J1 Conn_02x06_Odd_Even, J2 Conn_02x06_Odd_Even, J3 P1, J4 P2, J5 P3

Commit message: udated by FZ from Windows
Connections:
- net RXD: now reaches J1.7 (Pin_7)
- net TXD: now reaches J1.9 (Pin_9)
- no-connect marks 2 -> 0
