File: PCB/SIDE/SIDE.kicad_pcb (KiCad board)
At the start: 2 copper layers, 29 x 109 mm, 20 parts, among them IC1 VEML6030-GS15, J1 1_PIN, J2 1_PIN, J4 SM06B-SRSS-TB(LF)(SN), Q1 PJE8408_R1_00001, Q2 PJE8408_R1_00001, U1 AS7341DLG, U2 TMP112xxDRL

Commit message: udated by FZ from Windows
Parts:
- added U3: SHT4x, Sensor_Humidity:Sensirion_DFN-4_1.5x1.5mm_P0.8mm_SHT4x_NoCentralPad, F.Cu at (156.8, 95.5)
- U2: moved to B.Cu
- moved D2 27.9 mm to (153.5, 139.3), turned to -90 degrees
- moved R2 22.8 mm to (157.8, 72.7), turned to 90 degrees
- moved SC2 20.0 mm to (153.7, 132.0), turned to 180 degrees
- moved R3 17.1 mm to (157.8, 76.5), turned to 90 degrees
- moved IC1 13.3 mm to (160.9, 95.5)
- moved C1 11.2 mm to (158.6, 95.1), turned to 90 degrees
- moved U2 6.33 mm to (153.8, 94.7)
- moved R4 6.20 mm to (153.3, 91.6), turned to 90 degrees
- moved R5 5.12 mm to (156.7, 97.7), turned to 0 degrees
- moved U1 2.96 mm to (150.3, 95.5)
- moved C2 1.98 mm to (148.4, 96.0), turned to 0 degrees
- moved Q1 1.86 mm to (151.2, 92.9)
- moved R11 1.50 mm to (148.4, 93.8)
- moved D1 1.38 mm to (154.7, 52.0)
- moved Q2 0.85 mm to (149.5, 98.2)
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Routing:
- net /SC: track 0.00 -> 92.8 mm
- net /SCL: track 0.00 -> 53.1 mm, vias 0 -> 1
- net +3V3: track 0.00 -> 46.8 mm, vias 0 -> 5
- net +1V8: track 0.00 -> 42.9 mm, vias 0 -> 3
- net /SDA: track 0.00 -> 42.7 mm, vias 0 -> 1
- net Net-(IC1-ADDR): track 0.00 -> 5.35 mm, vias 0 -> 1
- net /SCL_1.8: track 0.00 -> 3.98 mm, vias 0 -> 1
- net /SDA_1.8: track 0.00 -> 2.78 mm, vias 0 -> 1
- net Net-(U2-ADD0): track 0.00 -> 1.47 mm
- net unconnected-(J2-Pad1): vias 0 -> 6
- net unconnected-(J1-Pad1): vias 0 -> 6
- net Net-(D2-A): vias 0 -> 13
- net Net-(D1-A): vias 0 -> 13
- net GND: vias 0 -> 64
- added copper zone on B.Cu, net GND
- added copper zone on F.Cu, net GND
- added copper zone on B.Cu, net Net-(D1-A)
- added copper zone on B.Cu, net Net-(D2-A)
- added copper zone on B.Cu, net unconnected-(J1-Pad1)
