File: PCB/SIDE/SIDE.kicad_sch (KiCad schematic)
At the start: 20 parts, among them IC1 VEML6030-GS15, J1 1_PIN, J2 1_PIN, J4 SM06B-SRSS-TB(LF)(SN), Q1 PJE8408_R1_00001, Q2 PJE8408_R1_00001, U1 AS7341DLG, U2 TMP112xxDRL

Commit message: udated by FZ from Windows
Parts:
- added U3: SHT4x, Sensor_Humidity:Sensirion_DFN-4_1.5x1.5mm_P0.8mm_SHT4x_NoCentralPad, symbol Sensor_Humidity:SHT4x
Connections:
- net +3V3: now also U3.3 (VDD)
- net GND: now also U3.4 (VSS)
- net SCL: now also U3.2 (SCL)
- net SDA: now also U3.1 (SDA)
Other:
- note added: "SHT4x"
- note added: "TMP112 - Body temperature"
- note removed: "TMP112"
- moved on the sheet: D1, D2, J1, J2, SC1, SC2
