File: PCB/SIDE/V3/SIDE.kicad_pcb (KiCad board)
At the start: 2 copper layers, 29 x 109 mm, 22 parts, among them IC1 VEML6030-GS15, J1 pin, J2 pin, J4 SM06B-SRSS-TB(LF)(SN), Q1 PJE8408_R1_00001, Q2 PJE8408_R1_00001, U1 AS7341DLG, U2 TMP112xxDRL, U3 SHT4x

Commit message: udated by FZ from Windows
Parts:
- removed D2: D_Schottky, Diode_SMD:D_0805_2012Metric_Pad1.15x1.40mm_HandSolder
Connections:
- SC1 pad 2: GND -> Net-(SC1--)
- SC2 pad 1: Net-(D2-A) -> Net-(SC1--)
Routing:
- net /SC: track 103.4 -> 19.6 mm
- net Net-(SC1--): track 0.00 -> 54.0 mm, vias 0 -> 19
- net Net-(D2-A): vias 13 -> 0
- added copper zone on B.Cu, net Net-(SC1--)
- removed copper zone on B.Cu, net Net-(D2-A)
