File: PCB/SIDE/V3/SIDE.kicad_sch (KiCad schematic)
At the start: 22 parts, among them IC1 VEML6030-GS15, J1 pin, J2 pin, J4 SM06B-SRSS-TB(LF)(SN), Q1 PJE8408_R1_00001, Q2 PJE8408_R1_00001, U1 AS7341DLG, U2 TMP112xxDRL, U3 SHT4x

Commit message: udated by FZ from Windows
Parts:
- removed D2: D_Schottky, Diode_SMD:D_0805_2012Metric_Pad1.15x1.40mm_HandSolder, symbol Device:D_Schottky
Connections:
- net GND: no longer SC1.2 (-)
- net at SC2.1 (+): now also SC1.2 (-)
Other:
- moved on the sheet: D1, SC1, SC2
Changed lines of the file:
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@@
   (junction (at 182.88 57.15) (diameter 0) (color 0 0 0 0)
-  )
-  (junction (at 107.95 97.79) (diameter 0) (color 0 0 0 0)
   )
   (junction (at 154.94 30.48) (diameter 0) (color 0 0 0 0)
@@
     (stroke (width 0) (type default))
   )
-  (wire (pts (xy 127 97.79) (xy 127 96.52))
+  (wire (pts (xy 125.73 96.52) (xy 125.73 97.79))
     (stroke (width 0) (type default))
   )
@@
     (stroke (width 0) (type default))
   )
-  (wire (pts (xy 107.95 78.74) (xy 127 78.74))
+  (wire (pts (xy 116.84 92.71) (xy 116.84 78.74))
     (stroke (width 0) (type default))
   )
@@
     (stroke (width 0) (type default))
   )
-  (wire (pts (xy 107.95 97.79) (xy 107.95 99.06))
-    (stroke (width 0) (type default))
-  )
   (polyline (pts (xy 13.97 138.43) (xy 13.97 107.95))
     (stroke (width 0) (type default))
   )
-  (wire (pts (xy 107.95 97.79) (xy 127 97.79))
-    (stroke (width 0) (type default))
-  )
   (wire (pts (xy 162.56 38.1) (xy 162.56 40.64))
     (stroke (width 0) (type default))
@@
     (stroke (width 0) (type default))
   )
-  (wire (pts (xy 127 87.63) (xy 127 88.9))
+  (wire (pts (xy 125.73 87.63) (xy 125.73 88.9))
     (stroke (width 0) (type default))
   )
@@
     (stroke (width 0) (type default))
   )
-  (wire (pts (xy 107.95 78.74) (xy 107.95 80.01))
+  (wire (pts (xy 109.22 82.55) (xy 109.22 83.82))
     (stroke (width 0) (type default))
   )
@@
     (stroke (width 0) (type default))
   )
-  (wire (pts (xy 127 78.74) (xy 127 80.01))
+  (wire (pts (xy 125.73 78.74) (xy 125.73 80.01))
     (stroke (width 0) (type default))
   )
@@
     (stroke (width 0) (type default))
   )
+  (wire (pts (xy 116.84 78.74) (xy 125.73 78.74))
+    (stroke (width 0) (type default))
+  )
   (wire (pts (xy 182.88 58.42) (xy 182.88 57.15))
     (stroke (width 0) (type default))
@@
     (stroke (width 0) (type default))
   )
-  (wire (pts (xy 107.95 87.63) (xy 107.95 88.9))
+  (wire (pts (xy 109.22 91.44) (xy 109.22 92.71))
     (stroke (width 0) (type default))
   )
@@
     (stroke (width 0) (type default))
   )
-  (wire (pts (xy 107.95 96.52) (xy 107.95 97.79))
-    (stroke (width 0) (type default))
-  )
   (polyline (pts (xy 143.51 71.12) (xy 180.34 71.12))
     (stroke (width 0) (type default))
@@
   )
   (wire (pts (xy 69.85 91.44) (xy 74.93 91.44))
+    (stroke (width 0) (type default))
+  )
+  (wire (pts (xy 109.22 92.71) (xy 116.84 92.71))
     (stroke (width 0) (type default))
   )
@@
     (effects (font (size 2.032 2.032) (thickness 0.3556) bold) (justify left bottom))
   )
-  (text "KXOB201K04F-TR" (at 109.22 96.52 0)
+  (text "KXOB201K04F-TR" (at 102.87 96.52 0)
     (effects (font (size 1.27 1.27)) (justify left bottom))
   )
@@
     (effects (font (size 1.27 1.27)) (justify left bottom))
   )
-  (label "SC" (at 115.57 78.74 0) (fields_autoplaced)
+  (label "SC" (at 109.22 82.55 0) (fields_autoplaced)
     (effects (font (size 1.27 1.27)) (justify left bottom))
   )
@@
     )
   )
-  (symbol (lib_id "Device:Solar_Cell") (at 127 93.98 0) (unit 1)
+  (symbol (lib_id "Device:Solar_Cell") (at 125.73 93.98 0) (unit 1)
     (in_bom yes) (on_board yes) (dnp no) (fields_autoplaced)
-    (property "Reference" "SC2" (at 129.667 90.797 0)
-      (effects (font (size 1.27 1.27)) (justify left))
-    )
-    (property "Value" "Solar_Cell" (at 129.667 92.845 0)
-      (effects (font (size 1.27 1.27)) (justify left))
-    )
-    (property "Footprint" "Mylib:KXOB201K04F-TR" (at 127 92.456 90)
-      (effects (font (size 1.27 1.27)) hide)
-    )
-    (property "Datasheet" "~" (at 127 92.456 90)
+    (property "Reference" "SC2" (at 128.397 90.797 0)
+      (effects (font (size 1.27 1.27)) (justify left))
+    )
+    (property "Value" "Solar_Cell" (at 128.397 92.845 0)
+      (effects (font (size 1.27 1.27)) (justify left))
+    )
+    (property "Footprint" "Mylib:KXOB201K04F-TR" (at 125.73 92.456 90)
+      (effects (font (size 1.27 1.27)) hide)
+    )
+    (property "Datasheet" "~" (at 125.73 92.456 90)
       (effects (font (size 1.27 1.27)) hide)
     )
@@
     )
   )
-  (symbol (lib_id "power:GND") (at 107.95 99.06 0) (unit 1)
+  (symbol (lib_id "power:GND") (at 125.73 97.79 0) (unit 1)
     (in_bom yes) (on_board yes) (dnp no) (fields_autoplaced)
-    (property "Reference" "#PWR06" (at 107.95 105.41 0)
-      (effects (font (size 1.27 1.27)) hide)
-    )
-    (property "Value" "GND" (at 107.95 103.5034 0)
-      (effects (font (size 1.27 1.27)))
-    )
-    (property "Footprint" "" (at 107.95 99.06 0)
-      (effects (font (size 1.27 1.27)) hide)
-    )
-    (property "Datasheet" "" (at 107.95 99.06 0)
+    (property "Reference" "#PWR06" (at 125.73 104.14 0)
+      (effects (font (size 1.27 1.27)) hide)
+    )
+    (property "Value" "GND" (at 125.73 102.2334 0)
+      (effects (font (size 1.27 1.27)))
+    )
+    (property "Footprint" "" (at 125.73 97.79 0)
+      (effects (font (size 1.27 1.27)) hide)
+    )
+    (property "Datasheet" "" (at 125.73 97.79 0)
       (effects (font (size 1.27 1.27)) hide)
     )
@@
     )
   )
-  (symbol (lib_id "Device:Solar_Cell") (at 107.95 93.98 0) (unit 1)
-    (in_bom yes) (on_board yes) (dnp no)
-    (property "Reference" "SC1" (at 110.617 90.797 0)
-      (effects (font (size 1.27 1.27)) (justify left))
-    )
-    (property "Value" "Solar_Cell" (at 110.617 92.845 0)
-      (effects (font (size 1.27 1.27)) (justify left))
-    )
-    (property "Footprint" "Mylib:KXOB201K04F-TR" (at 107.95 92.456 90)
-      (effects (font (size 1.27 1.27)) hide)
-    )
-    (property "Datasheet" "~" (at 107.95 92.456 90)
+  (symbol (lib_id "Device:Solar_Cell") (at 125.73 85.09 0) (unit 1)
+    (in_bom yes) (on_board yes) (dnp no)
+    (property "Reference" "SC1" (at 128.397 81.907 0)
+      (effects (font (size 1.27 1.27)) (justify left))
+    )
+    (property "Value" "Solar_Cell" (at 128.397 83.955 0)
+      (effects (font (size 1.27 1.27)) (justify left))
+    )
+    (property "Footprint" "Mylib:KXOB201K04F-TR" (at 125.73 83.566 90)
+      (effects (font (size 1.27 1.27)) hide)
+    )
+    (property "Datasheet" "~" (at 125.73 83.566 90)
       (effects (font (size 1.27 1.27)) hide)
     )
@@
         (path "/e63e39d7-6ac0-4ffd-8aa3-1841a4541b55"
           (reference "#PWR012") (unit 1)
-        )
-      )
-    )
-  )
-  (symbol (lib_id "Device:D_Schottky") (at 127 83.82 270) (unit 1)
-    (in_bom yes) (on_board yes) (dnp no) (fields_autoplaced)
-    (property "Reference" "D2" (at 129.032 83.5025 90)
-      (effects (font (size 1.27 1.27)) (justify left))
-    )
-    (property "Value" "D_Schottky" (at 124.968 82.4785 90)
-      (effects (font (size 1.27 1.27)) (justify right) hide)
-    )
-    (property "Footprint" "Diode_SMD:D_0805_2012Metric_Pad1.15x1.40mm_HandSolder" (at 127 83.82 0)
-      (effects (font (size 1.27 1.27)) hide)
-    )
-    (property "Datasheet" "~" (at 127 83.82 0)
-      (effects (font (size 1.27 1.27)) hide)
-    )
-    (pin "1")
-    (pin "2")
-    (instances
-      (project "SIDE"
-        (path "/e63e39d7-6ac0-4ffd-8aa3-1841a4541b55"
-          (reference "D2") (unit 1)
         )
       )
@@
     )
   )
-  (symbol (lib_id "Device:D_Schottky") (at 107.95 83.82 270) (unit 1)
+  (symbol (lib_id "Device:D_Schottky") (at 109.22 87.63 270) (unit 1)
     (in_bom yes) (on_board yes) (dnp no) (fields_autoplaced)
-    (property "Reference" "D1" (at 109.982 83.5025 90)
-      (effects (font (size 1.27 1.27)) (justify left))
-    )
-    (property "Value" "D_Schottky" (at 105.918 82.4785 90)
+    (property "Reference" "D1" (at 111.252 87.3125 90)
+      (effects (font (size 1.27 1.27)) (justify left))
+    )
+    (property "Value" "D_Schottky" (at 107.188 86.2885 90)
       (effects (font (size 1.27 1.27)) (justify right) hide)
     )
-    (property "Footprint" "Diode_SMD:D_0805_2012Metric_Pad1.15x1.40mm_HandSolder" (at 107.95 83.82 0)
-      (effects (font (size 1.27 1.27)) hide)
-    )
-    (property "Datasheet" "~" (at 107.95 83.82 0)
-      (effects (font (size 1.27 1.27)) hide)
-    )
+    (property "Footprint" "Diode_SMD:D_0805_2012Metric_Pad1.15x1.40mm_HandSolder" (at 109.22 87.63 0)
+      (effects (font (size 1.27 1.27)) hide)
+    )
+    (property "Datasheet" "~" (at 109.22 87.63 0)
+      (effects (font (size 1.27 1.27)) hide)
+    )
