File: PCB/PWR/V2/PWR.kicad_sch (KiCad schematic)
At the start: 39 parts, among them J1 Switch conn, J2 Conn_02x06_Odd_Even, J3 Battery, J4 Solar cell, U1 AP2112K-3.3, U2 BQ25570, U3 AP2112K-1.8, U4 MCP73831-2-OT

Commit message: udated by FZ from Windows
Parts:
- removed C1: 22uF, Capacitor_SMD:C_1206_3216Metric_Pad1.33x1.80mm_HandSolder, symbol Device:C_Small
- added R1: 1M, Resistor_SMD:R_1206_3216Metric_Pad1.30x1.75mm_HandSolder, symbol Device:R_Small
- R15: value 1k -> 10k
Connections:
- net GND: now also R1.1
- net VBAT: now also R1.2
Other:
- moved on the sheet: C10, C11, C12, C5, C9, J1, J3, J4, U1, U3
