File: PCB/DATA_STORAGE/DATA_STORAGE.kicad_pcb (KiCad board)
At the start: 2 copper layers, 40 x 46.2 mm, 3 parts, among them J1 Conn_02x06_Odd_Even, J2 Conn_02x06_Odd_Even

Commit message: udated by FZ from Windows
Parts:
- added C2: 0.1uF, Capacitor_SMD:C_0603_1608Metric_Pad1.08x0.95mm_HandSolder, F.Cu at (159.8, 90.7)
- added C3: 0.1uF, Capacitor_SMD:C_0603_1608Metric_Pad1.08x0.95mm_HandSolder, F.Cu at (145.9, 94.5)
- added IC1: CY15B108QN-40SXI, SamacSys_Parts:SOIC127P800X203-8N, F.Cu at (141.3, 98.7)
- added J3: 1660, SamacSys_Parts:1660, F.Cu at (160.4, 100.1)
- added Q1: DMG2305UX-7, SamacSys_Parts:SOT96P240X110-3N, B.Cu at (159.8, 97.3)
- added Q2: PJE8408_R1_00001, SamacSys_Parts:SOTFL50P160X60-3N, B.Cu at (156.5, 98.3)
- added R1: NC, Resistor_SMD:R_0603_1608Metric_Pad0.98x0.95mm_HandSolder, F.Cu at (150.0, 105.0)
- added R2: 10K, Resistor_SMD:R_0402_1005Metric_Pad0.72x0.64mm_HandSolder, F.Cu at (135.2, 99.3)
- added R3: 10k, Resistor_SMD:R_0603_1608Metric_Pad0.98x0.95mm_HandSolder, B.Cu at (166.0, 97.3)
Connections:
- J1 pad 7: unconnected-(J1-Pad7) -> /RXD
- J1 pad 9: unconnected-(J1-Pad9) -> /TXD
Routing:
- net VCC: track 3.41 -> 74.7 mm, vias 0 -> 1
- net /MISO: track 0.00 -> 42.8 mm, vias 0 -> 1
- net /SCK: track 0.00 -> 41.5 mm, vias 0 -> 1
- net /MOSI: track 0.00 -> 39.9 mm, vias 0 -> 1
- net /A5: track 0.00 -> 23.6 mm
- net /A1: track 0.00 -> 19.0 mm, vias 0 -> 1
- net Net-(J3-VDD): track 0.00 -> 11.2 mm, vias 0 -> 1
- net Net-(Q1-Pad1): track 0.00 -> 8.70 mm
- net /CARD_DETECT: track 0.00 -> 3.25 mm
- net GND: track 0.00 -> 3.13 mm, vias 0 -> 69
- net /~{WP}: track 0.00 -> 1.92 mm
- added copper zone on B.Cu, net GND
- added copper zone on F.Cu, net GND
Other:
- board text added: "Data_storage"
- board text added: "MIT MEDIA LAB RESENV"

Commit message: udated by FZ from Windows
Changed lines of the file:
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@@
     (grid_origin 150.16 123.198621)
     (pcbplotparams
-      (layerselection 0x0000020_7ffffffe)
+      (layerselection 0x00010fc_ffffffff)
       (plot_on_all_layers_selection 0x0000000_00000000)
       (disableapertmacros false)
@@
       (sketchpadsonfab false)
       (subtractmaskfromsilk false)
-      (outputformat 3)
+      (outputformat 1)
       (mirror false)
       (drillshape 0)
       (scaleselection 1)
-      (outputdirectory "")
+      (outputdirectory "Gerber/")
     )
   )
@@
     (fp_line (start 1 0.6) (end 1 -0.6)
       (stroke (width 0.1) (type solid)) (layer "F.Fab"))
-    (pad "1" smd roundrect (at -1.025 0 180) (size 1.15 1.4) (layers "F.Cu" "F.Paste" "F.Mask") (roundrect_rratio 0.217391)
+    (pad "1" smd roundrect (at -1.025 0 180) (size 1.15 1.4) (layers "F.Cu" "F.Paste" "F.Mask") (roundrect_rratio 0.2173913043)
       (net 2 "VCC") (pintype "passive"))
-    (pad "2" smd roundrect (at 1.025 0 180) (size 1.15 1.4) (layers "F.Cu" "F.Paste" "F.Mask") (roundrect_rratio 0.217391)
+    (pad "2" smd roundrect (at 1.025 0 180) (size 1.15 1.4) (layers "F.Cu" "F.Paste" "F.Mask") (roundrect_rratio 0.2173913043)
       (net 1 "GND") (pintype "passive"))
     (model "${KICAD6_3DMODEL_DIR}/LED_SMD.3dshapes/LED_0805_2012Metric.wrl"

Commit message: udated by FZ from Windows
Parts:
- removed C3: 0.1uF, Capacitor_SMD:C_0603_1608Metric_Pad1.08x0.95mm_HandSolder
- removed IC1: CY15B108QN-40SXI, SamacSys_Parts:SOIC127P800X203-8N
- removed R2: 10K, Resistor_SMD:R_0402_1005Metric_Pad0.72x0.64mm_HandSolder
- added C5: 0.1uF, Capacitor_SMD:C_0603_1608Metric_Pad1.08x0.95mm_HandSolder, F.Cu at (145.0, 94.9)
- added R4: 10K, Resistor_SMD:R_0603_1608Metric_Pad0.98x0.95mm_HandSolder, F.Cu at (135.1, 95.8)
- added R5: 10K, Resistor_SMD:R_0603_1608Metric_Pad0.98x0.95mm_HandSolder, F.Cu at (146.2, 97.5)
- added R6: 10K, Resistor_SMD:R_0603_1608Metric_Pad0.98x0.95mm_HandSolder, F.Cu at (136.7, 95.8)
- added U1: MB85RS2MT, Package_SO:SSOP-8_3.9x5.05mm_P1.27mm, F.Cu at (141.4, 98.7)
Routing:
- net /RXD: track 0.00 -> 19.0 mm, vias 0 -> 1
- net /~{WP}: track 1.92 -> 5.64 mm
- net VCC: track 74.7 -> 71.9 mm
- net /~{HL}: track 0.00 -> 2.29 mm
- net /SCK: track 41.5 -> 42.6 mm
- net /MISO: track 42.8 -> 42.0 mm
- net GND: vias 69 -> 67
