File: PCB/DATA_STORAGE/DATA_STORAGE.kicad_sch (KiCad schematic)
At the start: 4 parts, among them J1 Conn_02x06_Odd_Even, J2 Conn_02x06_Odd_Even

Commit message: udated by FZ from Windows
Parts:
- removed J?: 0473340001, 0473340001, symbol SamacSys_Legacy:0473340001
- added C2, C3: 0.1uF, Capacitor_SMD:C_0603_1608Metric_Pad1.08x0.95mm_HandSolder, symbol Device:C_Small
- added IC1: CY15B108QN-40SXI, SamacSys_Parts:SOIC127P800X203-8N, symbol SamacSys_Parts:CY15B108QN-40SXI
- added J3: 1660, SamacSys_Parts:1660, symbol SamacSys_Parts:1660
- added Q1: DMG2305UX-7, SamacSys_Parts:SOT96P240X110-3N, symbol SamacSys_Parts:DMG2305UX-7
- added Q2: PJE8408_R1_00001, SOTFL50P160X60-3N, symbol SamacSys_Parts:PJE8408_R1_00001
- added R1: NC, Resistor_SMD:R_0603_1608Metric_Pad0.98x0.95mm_HandSolder, symbol Device:R_Small
- added R2: 10K, Resistor_SMD:R_0402_1005Metric_Pad0.72x0.64mm_HandSolder, symbol Device:R_Small
- added R3: 10k, Resistor_SMD:R_0603_1608Metric_Pad0.98x0.95mm_HandSolder, symbol Device:R_Small
Connections:
- net A1: now also J3.2 (CD/DAT3)
- net A5: now also Q2.1
- net GND: now also C2.2, C3.1, IC1.4 (VSS), J3.11 (GND_1), J3.12 (GND_2), J3.6 (VSS), Q2.2
- net MISO: now also IC1.2 (SO), J3.7 (DAT0)
- net MOSI: now also IC1.5 (SI), J3.3 (CMD)
- net SCK: now also IC1.6 (SCK), J3.5 (CLK)
- net VCC: now also C2.1, C3.2, IC1.8 (VDD), Q1.2, R1.2, R2.2, R3.2
- net RXD: now reaches J1.7 (Pin_7)
- net TXD: now reaches J1.9 (Pin_9)
- new net: J3.4 (VDD), Q1.3
- new net: Q1.1, Q2.3, R3.1
- new net CARD_DETECT: J3.9 (CARD_DETECT_1), R1.1
- new net ~{FRAM_CS}: IC1.1 (~{CS})
- new net ~{WP}: IC1.3 (~{WP}), R2.1
- no-connect marks 2 -> 4
Other:
- note added: "Increase Arduino SD writing speed"
- note added: "https://arduino.stackexchange.com/questions/28540/how-to-increase-sd-card-write-speed-in-arduino"
- note added: "https://hackingmajenkoblog.wordpress.com/2016/03/25/fast-efficient-data-storage-on-an-arduino/"

Commit message: udated by FZ from Windows
Other:
- note added: "FRAM & SD card"
- note removed: "ADXL355 Module"
Changed lines of the file:
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@@
     (effects (font (size 1.35 1.35)) (justify left bottom))
   )
-  (text "ADXL355 Module" (at 16.51 21.59 0)
+  (text "FRAM & SD card" (at 16.51 21.59 0)
     (effects (font (size 3 3) (thickness 0.508) bold) (justify left bottom))
   )

Commit message: udated by FZ from Windows
Parts:
- removed C3: 0.1uF, Capacitor_SMD:C_0603_1608Metric_Pad1.08x0.95mm_HandSolder, symbol Device:C_Small
- removed IC1: CY15B108QN-40SXI, SamacSys_Parts:SOIC127P800X203-8N, symbol SamacSys_Parts:CY15B108QN-40SXI
- removed R2: 10K, Resistor_SMD:R_0402_1005Metric_Pad0.72x0.64mm_HandSolder, symbol Device:R_Small
- added C5: 0.1uF, Capacitor_SMD:C_0603_1608Metric_Pad1.08x0.95mm_HandSolder, symbol Device:C_Small
- added R4, R5, R6: 10K, Resistor_SMD:R_0603_1608Metric_Pad0.98x0.95mm_HandSolder, symbol Device:R_Small
- added U1: MB85RS2MT, Package_SO:SSOP-8_3.9x5.05mm_P1.27mm, symbol Memory_NVRAM:MB85RS2MT
- Q2: footprint SOTFL50P160X60-3N -> SamacSys_Parts:SOTFL50P160X60-3N
Connections:
- net GND: now also C5.1, U1.4 (GND)
- net MISO: now also U1.2 (SO)
- net MOSI: now also U1.5 (SI)
- net RXD: now also R6.1, U1.1 (~{CS})
- net SCK: now also U1.6 (SCK)
- net VCC: now also C5.2, R4.2, R5.2, R6.2, U1.8 (VDD)
- net ~{WP}: now also R4.1, U1.3 (~{WP})
- new net ~{HL}: R5.1, U1.7 (~{HOLD})
- no-connect marks 4 -> 3
