File: PCB/MCU/MCU.kicad_sch (KiCad schematic)
At the start: 36 parts, among them IC1 TMP112NAIDRLR, J1 Conn_02x06_Odd_Even, J2 Conn_02x06_Odd_Even, J3 USB_B_Micro, J4 Programmer, SW1 SW_Push, U1 MPU6050, U2 MDBT50Q-1MV2, U3 MAX6372, Y1 32.768kHz

Commit message: udated by FZ from Windows
Connections:
- net RXD: now reaches U2.48 (P0.24)
- net RXD: now also J1.7 (Pin_7)
- net TXD: now reaches U2.49 (P0.25)
- net TXD: now also J1.9 (Pin_9)
- no-connect marks 31 -> 27
Other:
- note added: "SSQ-106-03-T-D"
- note added: "SSQ-106-23-G-D"
- moved on the sheet: C9, J1, J2, J3, J4, R5, R6, TP1, TP2, TP3

Commit message: udated by FZ from Windows
Other:
- moved on the sheet: C9, J2, J3, J4, R5, R6, TP1, TP2, TP3

Commit message: udated by FZ from Windows
Parts:
- removed R3: 4.7K, Resistor_SMD:R_0603_1608Metric_Pad0.98x0.95mm_HandSolder, symbol Device:R_Small
- R11: value 120 -> 330
Connections:
- net ~{RESET}: now also U2.40 (P0.18/~{RESET})
Changed lines of the file:
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@@
+    (stroke (width 0) (type default))
+  )
+  (wire (pts (xy 26.67 82.55) (xy 40.64 82.55))
     (stroke (width 0) (type default))
   )
@@
     (stroke (width 0) (type default))
   )
-  (wire (pts (xy 22.86 82.55) (xy 30.48 82.55))
-    (stroke (width 0) (type default))
-  )
   (polyline (pts (xy 13.97 143.51) (xy 13.97 181.61))
     (stroke (width 0) (type default))
@@
   )
   (wire (pts (xy 190.5 34.29) (xy 191.77 34.29))
-    (stroke (width 0) (type default))
-  )
-  (wire (pts (xy 35.56 82.55) (xy 40.64 82.55))
     (stroke (width 0) (type default))
   )
@@
     (effects (font (size 1.27 1.27)) (justify left bottom))
   )
-  (label "~{RESET}" (at 22.86 82.55 0) (fields_autoplaced)
+  (label "~{RESET}" (at 26.67 82.55 0) (fields_autoplaced)
     (effects (font (size 1.27 1.27)) (justify left bottom))
   )
@@
       (effects (font (size 1.27 1.27)))
     )
-    (property "Value" "120" (at 107.95 134.112 90)
+    (property "Value" "330" (at 107.95 134.112 90)
       (effects (font (size 1.27 1.27)))
     )
@@
         )
       )
-    )
-  )
-  (symbol (lib_id "Device:R_Small") (at 33.02 82.55 270) (unit 1)
-    (in_bom yes) (on_board yes) (dnp no)
-    (property "Reference" "R3" (at 33.02 84.328 90)
-      (effects (font (size 1.27 1.27)))
-    )
-    (property "Value" "4.7K" (at 33.02 80.518 90)
-      (effects (font (size 1.27 1.27)))
-    )
-    (property "Footprint" "Resistor_SMD:R_0603_1608Metric_Pad0.98x0.95mm_HandSolder" (at 33.02 82.55 0)
-      (effects (font (size 1.27 1.27)) hide)
-    )
-    (property "Datasheet" "~" (at 33.02 82.55 0)
-      (effects (font (size 1.27 1.27)) hide)
-    )
-    (pin "1")
-    (pin "2")
-    (instances
-      (project "MCU"
-        (path "/e63e39d7-6ac0-4ffd-8aa3-1841a4541b55"
-          (reference "R3") (unit 1)
-        )
-      )

Commit message: udated by FZ from Windows
Changed lines of the file:
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@@
     (effects (font (size 1.27 1.27)) (justify right bottom))
   )
-  (label "MOSI" (at 34.29 69.85 180) (fields_autoplaced)
-    (effects (font (size 1.27 1.27)) (justify right bottom))
+  (label "MOSI" (at 34.29 69.85 0) (fields_autoplaced)
+    (effects (font (size 1.27 1.27)) (justify left bottom))
   )
   (label "D6" (at 34.29 54.61 0) (fields_autoplaced)
