File: PCB/CONN/CONN.kicad_sch (KiCad schematic)
At the start: 25 parts, among them J1 Conn_02x06_Odd_Even, J2 Solar cell, J3 Conn_02x06_Odd_Even, J4 BM06B-SURS-TF(LF)(SN), J5 BM06B-SURS-TF(LF)(SN), J6 BM06B-SURS-TF(LF)(SN), J8 BM06B-SURS-TF(LF)(SN), J9 BM06B-SURS-TF(LF)(SN), U1 TCA9548APWR

Commit message: udated by FZ from Windows
Parts:
- J4, J5, J6, J8, J9: value BM06B-SURS-TF(LF)(SN) -> BM06B-SRSS-TBT(LF)(SN)
- J7: value (none) -> BM06B-SRSS-TBT(LF)(SN)

Commit message: udated by FZ from Windows
Other:
- moved on the sheet: J5, J6, J7

Commit message: udated by FZ from Windows
Other:
- note added: "I2C addr = 0x70"
Changed lines of the file:
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@@
+    (effects (font (size 1.27 1.27)) (justify left bottom))
+  )
+  (text "I2C addr = 0x70" (at 22.86 78.74 0)
     (effects (font (size 1.27 1.27)) (justify left bottom))
   )
