File: PCB/BURNING_R/V1/BURNING_R.kicad_pcb (KiCad board)
At the start: 2 copper layers, 40 x 46.2 mm, 32 parts, among them J1 Conn_02x06_Odd_Even, J2 Conn_02x06_Odd_Even, J3 BR_conn, J4 BR_conn, J5 BR_conn, J6 BR_conn, J7 BR_conn, J8 BR_conn, J9 Battery, Q1 DMN2056U-7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

Commit message: udated by FZ from Windows
Parts:
- C4: footprint Capacitor_SMD:C_0402_1005Metric_Pad0.74x0.62mm_HandSolder -> Capacitor_SMD:C_0603_1608Metric_Pad1.08x0.95mm_HandSolder
- Q1: value DMN2056U-7 -> DMN2056U
- Q2, Q3, Q4, Q5, Q6: value NMOS -> DMN2056U
- R10, R11, R4, R5, R6, R7, R8, R9: footprint Resistor_SMD:R_0402_1005Metric_Pad0.72x0.64mm_HandSolder -> Resistor_SMD:R_0603_1608Metric_Pad0.98x0.95mm_HandSolder
- R2: value 100 -> 1k
- moved R10 2.20 mm to (146.3, 101.8)
- moved R11 2.20 mm to (138.4, 101.8)
- moved R9 2.18 mm to (154.2, 101.8)
- moved R8 1.56 mm to (140.3, 98.7)
- moved R6 1.54 mm to (156.1, 98.7)
- moved R7 1.48 mm to (148.1, 98.6)
- moved R5 1.37 mm to (157.3, 89.4)
- moved R4 0.33 mm to (153.6, 89.4)
- moved C4 0.33 mm to (145.8, 89.5)
- moved Q6 0.10 mm to (156.0, 97.7), turned to 180 degrees
- moved Q4 0.10 mm to (140.2, 97.7), turned to 180 degrees
- moved Q5 0.10 mm to (148.1, 97.7), turned to 180 degrees
- turned Q1 to 0 degrees
- turned Q3 to 0 degrees
- turned Q2 to 0 degrees
Connections:
- Q1 pad 1: /BR_1 -> /BR_1_EN
- Q1 pad 2: /BR_1_EN -> GND
- Q1 pad 3: GND -> /BR_1
- Q2 pad 1: /BR_2 -> /BR_2_EN
- Q2 pad 2: /BR_2_EN -> GND
- Q2 pad 3: GND -> /BR_2
- Q3 pad 1: /BR_3 -> /BR_3_EN
- Q3 pad 2: /BR_3_EN -> GND
- Q3 pad 3: GND -> /BR_3
- Q4 pad 1: /BR_4 -> /BR_4_EN
- Q4 pad 2: /BR_4_EN -> GND
- Q4 pad 3: GND -> /BR_4
- Q5 pad 1: /BR_5 -> /BR_5_EN
- Q5 pad 2: /BR_5_EN -> GND
- Q5 pad 3: GND -> /BR_5
- Q6 pad 1: /BR_6 -> /BR_6_EN
- Q6 pad 2: /BR_6_EN -> GND
- Q6 pad 3: GND -> /BR_6
Routing:
- net /BR_6_EN: track 12.9 -> 10.2 mm
- net /BR_1_EN: track 27.8 -> 29.7 mm
- net /BR_2_EN: track 19.2 -> 21.1 mm
- net /BR_3_EN: track 7.62 -> 9.49 mm
- net /BR_4_EN: track 27.1 -> 25.2 mm
- net /BR_5_EN: track 20.9 -> 19.1 mm
- net /SCL: track 24.3 -> 23.6 mm
- net /SDA: track 17.4 -> 18.1 mm
- net GND: vias 105 -> 103
