File: PCB/BURNING_R/V1/BURNING_R.kicad_sch (KiCad schematic)
At the start: 32 parts, among them J1 Conn_02x06_Odd_Even, J2 Conn_02x06_Odd_Even, J3 BR_conn, J4 BR_conn, J5 BR_conn, J6 BR_conn, J7 BR_conn, J8 BR_conn, J9 Battery, Q1 DMN2056U-7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

Commit message: udated by FZ from Windows
Parts:
- removed Q1: DMN2056U-7, Package_TO_SOT_SMD:SOT-23, symbol Simulation_SPICE:NMOS
- removed Q2, Q3, Q4, Q5, Q6: NMOS, Package_TO_SOT_SMD:SOT-23, symbol Simulation_SPICE:NMOS
- added Q1, Q2, Q3, Q4, Q5, Q6: DMN2056U, Package_TO_SOT_SMD:SOT-23, symbol Transistor_FET:DMN2056U
- C13: footprint Capacitor_SMD:C_0402_1005Metric_Pad0.74x0.62mm_HandSolder -> Capacitor_SMD:C_0603_1608Metric_Pad1.08x0.95mm_HandSolder
- R10, R11, R4, R5, R6, R7, R8, R9: footprint Resistor_SMD:R_0402_1005Metric_Pad0.72x0.64mm_HandSolder -> Resistor_SMD:R_0603_1608Metric_Pad0.98x0.95mm_HandSolder
- R16: value 100 -> 1k
Connections:
- net BR_1: now also Q1.3 (D)
- net BR_1_EN: now also Q1.1 (G)
- net BR_2: now also Q2.3 (D)
- net BR_2_EN: now also Q2.1 (G)
- net BR_3: now also Q3.3 (D)
- net BR_3_EN: now also Q3.1 (G)
- net BR_4: now also Q4.3 (D)
- net BR_4_EN: now also Q4.1 (G)
- net BR_5: now also Q5.3 (D)
- net BR_5_EN: now also Q5.1 (G)
- net BR_6: now also Q6.3 (D)
- net BR_6_EN: now also Q6.1 (G)
- net GND: now also Q1.2 (S), Q2.2 (S), Q3.2 (S), Q4.2 (S), Q5.2 (S), Q6.2 (S)
Other:
- note added: "CH_0"
- note added: "CH_1"
- note added: "CH_2"
- note added: "CH_3"
- note added: "CH_4"
- note added: "CH_5"
